Commit message: fixing urdf joint limits

File: phantom_touch_description/urdf/phantom_touch.urdf (robot description, URDF)
Before this commit: robot phantom_touch, 9 links, 8 joints
Links:
- removed link base_bottom
- removed link stylus_point
- link base: geometry visual mesh filename=package://omni_description/meshes/base.stl
- link lower_arm: geometry visual mesh filename=package://omni_description/meshes/lower_arm.stl
- link stylus: geometry visual mesh filename=package://omni_description/meshes/pen.stl
- link tip: geometry visual mesh filename=package://omni_description/meshes/tip.stl
- link torso: geometry visual mesh filename=package://omni_description/meshes/torso.stl
- link upper_arm: geometry visual mesh filename=package://omni_description/meshes/upper_arm.stl
- link wrist: geometry visual mesh filename=package://omni_description/meshes/wrist.stl
Joints:
- removed joint connector_joint
- removed joint stylus_point_joint
- joint elbow: limit lower=-0.81 upper=1.25 effort=5 velocity=100 -> lower=-0.83 upper=1.19 effort=5 velocity=100
- joint pitch: limit lower=-0.5 upper=1.75 effort=5 velocity=100 -> lower=-1.431 upper=1.081 effort=5 velocity=100
- joint roll: limit lower=-2.58 upper=2.58 effort=5 velocity=100 -> lower=-2.617 upper=2.613 effort=5 velocity=100; origin xyz=0 -0.023 0 rpy=-3.14159 3.14159 0 -> xyz=0 -0.023 0 rpy=3.14159 3.14159 0
- joint shoulder: limit lower=0 upper=1.75 effort=5 velocity=100 -> lower=-0.028 upper=1.787 effort=5 velocity=100
- joint waist: parent base_bottom -> base
- joint yaw: limit lower=3.92 upper=8.83 effort=5 velocity=100 -> lower=-2.55 upper=2.57 effort=5 velocity=100
